Commit message: Collision between collidable box and Mls is working now

File: src/smurf/just_a_box/urdf/just_a_box.urdf (robot description, URDF)
Before this commit: robot just_a_box, 2 links, 1 joints
Links:
- removed link root
- link box: geometry collision box size=1.0 1.0 1.0; visual box size=1.0 1.0 1.0
Joints:
- removed joint root2box
