Commit message: Test for collisions with multiple types of objects is working

File: src/smurf/multiple_objects/urdf/multiple_objects.urdf (robot description, URDF)
Before this commit: robot multiple_objects, 1 links, 0 joints
Links:
- added link sphere, mass 1.121; collision sphere radius=0.5; visual sphere radius=0.5
Joints:
- added joint box2sphere: type fixed, parent box, child sphere, origin xyz=3.0 3.0 3.0 rpy=0 0 0, axis 0.0 0.0 0, limit lower=-0.785398 upper=0.785398 effort=1000 velocity=6.28
